Commit message: fk working

File: interbotix_descriptions/urdf/rx200.urdf (robot description, URDF)
Before this commit: robot rx200, 13 links, 12 joints
Links:
- link /base_link: mass 0.766135 -> 1.0
- link /ee_arm_link: mass 0.001 -> 0.00001
- link /ee_gripper_link: mass 0.001 -> 0.00001
- link /fingers_link: mass 0.001 -> 0.00001
- link /forearm_link: mass 0.258863 -> 0.00001
- link /gripper_bar_link: mass 0.034199 -> 0.00001
- link /gripper_link: mass 0.072885 -> 0.00001
- link /gripper_prop_link: mass 0.00434 -> 0.00001
- link /left_finger_link: mass 0.016246 -> 0.00001
- link /right_finger_link: mass 0.016246 -> 0.00001
- link /shoulder_link: mass 0.257774 -> 0.00001
- link /upper_arm_link: mass 0.297782 -> 0.00001
- link /wrist_link: mass 0.084957 -> 0.00001

Commit message: ik fully working. yet to test on rx200

File: interbotix_descriptions/urdf/rx200.urdf (robot description, URDF)
Before this commit: robot rx200, 13 links, 12 joints
Links:
- link /base_link: mass 1.0 -> 1
- link /ee_arm_link: mass 0.00001 -> 0.000010001
- link /ee_gripper_link: mass 0.00001 -> 0.000010001
- link /fingers_link: mass 0.00001 -> 0.000010001
- link /forearm_link: mass 0.00001 -> 0.000010001
- link /gripper_bar_link: mass 0.00001 -> 0.000010001
- link /gripper_link: mass 0.00001 -> 0.000010001
- link /gripper_prop_link: mass 0.00001 -> 0.000010001
- link /left_finger_link: mass 0.00001 -> 0.000010001
- link /right_finger_link: mass 0.00001 -> 0.000010001
- link /shoulder_link: mass 0.00001 -> 0.000010001
- link /upper_arm_link: mass 0.00001 -> 0.000010001
- link /wrist_link: mass 0.00001 -> 0.000010001

File: models/dof.urdf (robot description, URDF)
Before this commit: robot morpheus, 7 links, 6 joints
Links:
- added link j4, mass .000000001; collision cylinder length=0.1 radius=0.05; visual cylinder length=0.1 radius=0.05
- added link j5, mass .000000001; collision cylinder length=0.1 radius=0.05; visual cylinder length=0.1 radius=0.05
- added link j6, mass .000000001; collision cylinder length=0.1 radius=0.05; visual cylinder length=0.1 radius=0.05
- added link l4, mass .000000001; collision box size=0.05 0.05 0.125; visual box size=0.05 0.05 0.125
- added link l5, mass .000000001; collision box size=0.05 0.05 0.125; visual box size=0.05 0.05 0.125
- added link l6, mass .000000001; collision box size=0.05 0.05 0.125; visual box size=0.05 0.05 0.125
Joints:
- removed joint phalange_to_ee
- added joint j4_to_l4: type revolute, parent j4, child l4, origin xyz=0 0 0 rpy=0 0 0, axis 1 0 0, limit lower=-3.1415 upper=3.1415 effort=10 velocity=0.25
- added joint j4_to_l5: type revolute, parent j5, child l5, origin xyz=0 0 0 rpy=0 0 0, axis 0 1 0, limit lower=-3.1415 upper=3.1415 effort=10 velocity=0.25
- added joint j6_to_l6: type revolute, parent j6, child l6, origin xyz=0 0 0 rpy=0 0 0, axis 1 0 0, limit lower=-3.1415 upper=3.1415 effort=10 velocity=0.25
- added joint l4_to_j5: type fixed, parent l4, child j5, origin xyz=0.125 0 0 rpy=0 0 0, axis 0 0 1
- added joint l5_to_j6: type fixed, parent l5, child j6, origin xyz=0.125 0 0 rpy=0 0 0, axis 0 0 1
- added joint l6_to_ee: type fixed, parent l6, child ee, origin xyz=0.125 0 0 rpy=0 0 0
- added joint phalange_to_j4: type fixed, parent phalange, child j4, origin xyz=0.5 0. 0.0 rpy=0 0 0
- joint carpal_to_phalange: origin xyz=0 0. 0.0 rpy=0 0 0 -> xyz=0 0 0 rpy=0 0 0

Commit message: wrist center spatial ik implemented

File: interbotix_descriptions/urdf/rx200.urdf (robot description, URDF)
Before this commit: robot rx200, 13 links, 12 joints
Joints:
- joint elbow: origin xyz=0.05 0 0.2 rpy=3.14159265359 0 0 -> xyz=0.05 0 0.2 rpy=3.14159265359 0.3084 0
- joint shoulder: origin xyz=0 0 0.03891 rpy=0 0 0 -> xyz=0 0 0.03891 rpy=0 -0.23 0
